Commit message: 搭建vi_car仿真小车URDF：差速四轮(25x10cm,轮径5cm)+2D雷达+IMU+全套Gazebo插件

File: urdf/vi_car.urdf (robot description, URDF)
Before this commit: robot vi_car, 4 links, 3 joints
Links:
- removed link camera_link
- added link base_footprint
- added link left_front_wheel, mass 0.05; collision cylinder length=0.025 radius=0.025; visual cylinder length=0.025 radius=0.025
- added link left_rear_wheel, mass 0.05; collision cylinder length=0.025 radius=0.025; visual cylinder length=0.025 radius=0.025
- added link lidar_mount, mass 0.03; collision cylinder length=0.05 radius=0.012; visual cylinder length=0.05 radius=0.012
- added link right_front_wheel, mass 0.05; collision cylinder length=0.025 radius=0.025; visual cylinder length=0.025 radius=0.025
- added link right_rear_wheel, mass 0.05; collision cylinder length=0.025 radius=0.025; visual cylinder length=0.025 radius=0.025
- link base_link: mass None -> 0.6; geometry collision box size=0.25 0.10 0.02; visual box size=0.25 0.10 0.02
- link imu_link: mass None -> 0.01; geometry collision box size=0.015 0.015 0.005; visual box size=0.015 0.015 0.005
- link laser_link: mass None -> 0.05; geometry collision cylinder length=0.04 radius=0.035; visual cylinder length=0.04 radius=0.035
Joints:
- removed joint base_to_camera
- removed joint base_to_imu
- removed joint base_to_laser
- added joint base_joint: type fixed, parent base_footprint, child base_link, origin xyz=0 0 0.025 rpy=0 0 0
- added joint imu_joint: type fixed, parent base_link, child imu_link, origin xyz=-0.03 0 0.0125 rpy=0 0 0
- added joint laser_joint: type fixed, parent lidar_mount, child laser_link, origin xyz=0 0 0.045 rpy=0 0 0
- added joint left_front_wheel_joint: type continuous, parent base_link, child left_front_wheel, origin xyz=0.075 0.0625 0 rpy=0 0 0, axis 0 1 0
- added joint left_rear_wheel_joint: type continuous, parent base_link, child left_rear_wheel, origin xyz=-0.075 0.0625 0 rpy=0 0 0, axis 0 1 0
- added joint lidar_mount_joint: type fixed, parent base_link, child lidar_mount, origin xyz=0 0 0.035 rpy=0 0 0
- added joint right_front_wheel_joint: type continuous, parent base_link, child right_front_wheel, origin xyz=0.075 -0.0625 0 rpy=0 0 0, axis 0 1 0
- added joint right_rear_wheel_joint: type continuous, parent base_link, child right_rear_wheel, origin xyz=-0.075 -0.0625 0 rpy=0 0 0, axis 0 1 0
